File: boards/rgbdriver/rgbdriver.sch (KiCad schematic (older format))
At the start: 7 parts, among them U1 rgb.breakout

Commit message: updated pcb
Parts:
- R1, R3: footprint (none) -> Resistors_ThroughHole:Resistor_Horizontal_RM10mm
Changed lines of the file:
@@
 F 0 "R1" V 3680 2350 50  0000 C CNN
 F 1 "10k" V 3600 2350 50  0000 C CNN
-F 2 "" V 3530 2350 50  0001 C CNN
+F 2 "Resistors_ThroughHole:Resistor_Horizontal_RM10mm" V 3530 2350 50  0001 C CNN
 F 3 "" H 3600 2350 50  0000 C CNN
 	1    3600 2350
@@
 F 0 "R3" V 6930 2350 50  0000 C CNN
 F 1 "10k" V 6850 2350 50  0000 C CNN
-F 2 "" V 6780 2350 50  0001 C CNN
+F 2 "Resistors_ThroughHole:Resistor_Horizontal_RM10mm" V 6780 2350 50  0001 C CNN
 F 3 "" H 6850 2350 50  0000 C CNN
 	1    6850 2350
