File: boards/led/led.sch (KiCad schematic (older format))
At the start: 2 parts, among them J1 RJ45

Commit message: another revision
Parts:
- added P1: CONN_01X08, Pin_Headers:Pin_Header_Straight_1x08, symbol CONN_01X08
Connections:
- net at D1.1 (RC), J1.1: now also P1.1 (P1)
- net at D1.2 (GC), J1.3: now also P1.3 (P3)
- net at D1.3 (BC), J1.5: now also P1.5 (P5)
- net at D1.4 (BA), J1.6: now also P1.6 (P6)
- net at D1.5 (GA), J1.4: now also P1.4 (P4)
- net at D1.6 (RA), J1.2: now also P1.2 (P2)
- net at J1.7: now also P1.7 (P7)
- net at J1.8: now also P1.8 (P8)
- no-connect marks 3 -> 1
Changed lines of the file:
@@
 $EndComp
 Wire Wire Line
-	4700 3150 4700 3700
+	4700 1950 4700 3700
 Wire Wire Line
 	4700 3700 4850 3700
 Wire Wire Line
-	4800 3150 4800 3400
+	4800 1950 4800 3400
 Wire Wire Line
 	4800 3400 5250 3400
@@
 	5250 3400 5250 3700
 Wire Wire Line
-	4900 3150 4900 3250
+	4900 1950 4900 3250
 Wire Wire Line
 	4900 3250 4550 3250
@@
 	4550 3900 4850 3900
 Wire Wire Line
-	5000 3150 5000 3350
+	5000 1950 5000 3350
 Wire Wire Line
 	5000 3350 5300 3350
@@
 	5300 3900 5250 3900
 Wire Wire Line
-	5100 3150 5100 3300
+	5100 1950 5100 3300
 Wire Wire Line
 	5100 3300 4500 3300
@@
 	4500 4100 4850 4100
 Wire Wire Line
-	5200 3150 5200 3300
+	5200 1950 5200 3300
 Wire Wire Line
 	5200 3300 5350 3300
@@
 	5350 4100 5250 4100
 NoConn ~ 5600 2350
-NoConn ~ 5300 3150
-NoConn ~ 5400 3150
+$Comp
+L CONN_01X08 P1
+U 1 1 578D0BE9
+P 5050 1750
+F 0 "P1" H 5050 2200 50  0000 C CNN
+F 1 "CONN_01X08" V 5150 1750 50  0000 C CNN
+F 2 "Pin_Headers:Pin_Header_Straight_1x08" H 5050 1750 50  0000 C CNN
+F 3 "" H 5050 1750 50  0000 C CNN
+	1    5050 1750
+	0    -1   -1   0
+$EndComp
+Connection ~ 4700 3150
+Connection ~ 4800 3150
+Connection ~ 4900 3150
+Connection ~ 5000 3150
+Connection ~ 5100 3150
+Connection ~ 5200 3150
+Wire Wire Line
+	5300 3150 5300 1950
+Wire Wire Line
+	5400 3150 5400 1950
 $EndSCHEMATC
