File: boards/motherboard/motherboard.kicad_pcb (KiCad board)
At the start: 2 copper layers, 214.4 x 64 mm, 50 parts, among them CN1 CONN_01X02, CN2 CONN_01X02, CN3 CONN_01X02, CN4 CONN_01X02, CN5 CONN_01X02, J1 RJ45, J2 RJ45, J3 RJ45, J4 RJ45, J5 RJ45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

Commit message: minor tweaks
Routing:
- net VCC: track 295.5 -> 302.5 mm
Changed lines of the file:
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@@
   (segment (start 229.848 63.8021) (end 236.22 62.23) (width 0.25) (layer B.Cu) (net 6))
   (segment (start 226.2929 63.8021) (end 229.848 63.8021) (width 0.25) (layer B.Cu) (net 6))
-  (segment (start 224.627 65.468) (end 226.2929 63.8021) (width 0.25) (layer B.Cu) (net 6))
-  (segment (start 224.627 68.362) (end 224.627 65.468) (width 0.25) (layer B.Cu) (net 6))
+  (segment (start 226.314 65.532) (end 226.2929 63.8021) (width 0.25) (layer B.Cu) (net 6))
+  (segment (start 224.627 68.362) (end 226.314 65.532) (width 0.25) (layer B.Cu) (net 6))
   (segment (start 223.139 90.17) (end 222.885 90.17) (width 0.4) (layer F.Cu) (net 7))
   (segment (start 222.885 90.17) (end 219.964 93.091) (width 0.4) (layer F.Cu) (net 7))
@@
   (segment (start 177.292 76.454) (end 166.37 76.454) (width 0.25) (layer F.Cu) (net 47))
   (segment (start 178.054 77.216) (end 177.292 76.454) (width 0.25) (layer F.Cu) (net 47))
-  (segment (start 64.9499 77.3959) (end 66.294 78.74) (width 0.25) (layer F.Cu) (net 47))
-  (segment (start 51.054 78.74) (end 52.3981 77.3959) (width 0.25) (layer F.Cu) (net 47))
-  (segment (start 52.3981 77.3959) (end 64.9499 77.3959) (width 0.25) (layer F.Cu) (net 47))
-  (segment (start 108.204 78.74) (end 109.5289 77.4151) (width 0.25) (layer F.Cu) (net 47))
-  (segment (start 120.8491 77.4151) (end 109.5289 77.4151) (width 0.25) (layer F.Cu) (net 47))
-  (segment (start 122.174 78.74) (end 120.8491 77.4151) (width 0.25) (layer F.Cu) (net 47))
-  (segment (start 92.9091 77.4151) (end 94.234 78.74) (width 0.25) (layer F.Cu) (net 47))
-  (segment (start 81.5889 77.4151) (end 92.9091 77.4151) (width 0.25) (layer F.Cu) (net 47))
-  (segment (start 80.264 78.74) (end 81.5889 77.4151) (width 0.25) (layer F.Cu) (net 47))
-  (segment (start 95.5589 77.4151) (end 94.234 78.74) (width 0.25) (layer F.Cu) (net 47))
-  (segment (start 109.5289 77.4151) (end 95.5589 77.4151) (width 0.25) (layer F.Cu) (net 47))
-  (segment (start 123.5424 80.1084) (end 122.174 78.74) (width 0.25) (layer B.Cu) (net 47))
-  (segment (start 134.7756 80.1084) (end 123.5424 80.1084) (width 0.25) (layer B.Cu) (net 47))
-  (segment (start 136.144 78.74) (end 134.7756 80.1084) (width 0.25) (layer B.Cu) (net 47))
-  (segment (start 148.771 80.083) (end 150.114 78.74) (width 0.25) (layer B.Cu) (net 47))
-  (segment (start 137.487 80.083) (end 148.771 80.083) (width 0.25) (layer B.Cu) (net 47))
-  (segment (start 136.144 78.74) (end 137.487 80.083) (width 0.25) (layer B.Cu) (net 47))
-  (segment (start 162.6733 80.1507) (end 164.084 78.74) (width 0.25) (layer B.Cu) (net 47))
-  (segment (start 150.114 78.74) (end 151.5247 80.1507) (width 0.25) (layer B.Cu) (net 47))
-  (segment (start 151.5247 80.1507) (end 162.6733 80.1507) (width 0.25) (layer B.Cu) (net 47))
-  (segment (start 205.994 80.0781) (end 205.994 78.74) (width 0.25) (layer F.Cu) (net 47))
-  (segment (start 218.6259 80.0781) (end 205.994 80.0781) (width 0.25) (layer F.Cu) (net 47))
-  (segment (start 219.964 78.74) (end 218.6259 80.0781) (width 0.25) (layer F.Cu) (net 47))
-  (segment (start 193.3621 80.0781) (end 192.024 78.74) (width 0.25) (layer F.Cu) (net 47))
-  (segment (start 205.994 80.0781) (end 193.3621 80.0781) (width 0.25) (layer F.Cu) (net 47))
+  (segment (start 65.024 76.962) (end 66.294 78.74) (width 0.25) (layer F.Cu) (net 47))
+  (segment (start 51.054 78.74) (end 52.832 76.962) (width 0.25) (layer F.Cu) (net 47))
+  (segment (start 52.832 76.962) (end 65.024 76.962) (width 0.25) (layer F.Cu) (net 47))
+  (segment (start 108.204 78.74) (end 109.474 76.962) (width 0.25) (layer F.Cu) (net 47))
+  (segment (start 120.65 76.962) (end 109.474 76.962) (width 0.25) (layer F.Cu) (net 47))
+  (segment (start 122.174 78.74) (end 120.65 76.962) (width 0.25) (layer F.Cu) (net 47))
+  (segment (start 92.964 76.962) (end 94.234 78.74) (width 0.25) (layer F.Cu) (net 47))
+  (segment (start 81.534 76.962) (end 92.964 76.962) (width 0.25) (layer F.Cu) (net 47))
+  (segment (start 80.264 78.74) (end 81.534 76.962) (width 0.25) (layer F.Cu) (net 47))
+  (segment (start 95.758 76.962) (end 94.234 78.74) (width 0.25) (layer F.Cu) (net 47))
+  (segment (start 109.474 76.962) (end 95.758 76.962) (width 0.25) (layer F.Cu) (net 47))
+  (segment (start 123.698 80.772) (end 122.174 78.74) (width 0.25) (layer B.Cu) (net 47))
+  (segment (start 134.874 80.772) (end 123.698 80.772) (width 0.25) (layer B.Cu) (net 47))
+  (segment (start 136.144 78.74) (end 134.874 80.772) (width 0.25) (layer B.Cu) (net 47))
+  (segment (start 148.844 80.772) (end 150.114 78.74) (width 0.25) (layer B.Cu) (net 47))
+  (segment (start 137.414 80.772) (end 148.844 80.772) (width 0.25) (layer B.Cu) (net 47))
+  (segment (start 136.144 78.74) (end 137.414 80.772) (width 0.25) (layer B.Cu) (net 47))
+  (segment (start 162.306 80.772) (end 164.084 78.74) (width 0.25) (layer B.Cu) (net 47))
+  (segment (start 150.114 78.74) (end 151.384 80.772) (width 0.25) (layer B.Cu) (net 47))
+  (segment (start 151.384 80.772) (end 162.306 80.772) (width 0.25) (layer B.Cu) (net 47))
+  (segment (start 205.994 80.772) (end 205.994 78.74) (width 0.25) (layer F.Cu) (net 47))
+  (segment (start 218.694 80.772) (end 205.994 80.772) (width 0.25) (layer F.Cu) (net 47))
+  (segment (start 219.964 78.74) (end 218.694 80.772) (width 0.25) (layer F.Cu) (net 47))
+  (segment (start 193.294 80.772) (end 192.024 78.74) (width 0.25) (layer F.Cu) (net 47))
+  (segment (start 205.994 80.772) (end 193.294 80.772) (width 0.25) (layer F.Cu) (net 47))
   (segment (start 242.824 97.028) (end 243.586 97.028) (width 0.25) (layer F.Cu) (net 50))
   (segment (start 243.586 97.028) (end 245.618 94.996) (width 0.25) (layer F.Cu) (net 50))
