File: boards/magicstick/magicstick.sch (KiCad schematic (older format))
At the start: 16 parts

Commit message: magic stick circuit
Parts:
- added D?: LED_RCBG, symbol LED_RCBG
- added R?: 32, symbol R
- added R? (x2): 21, symbol R
- added RFID?: RFID-RC522, symbol RFID-RC522
- added U?: NodeMCU_Amica_R2, symbol NodeMCU_Amica_R2
Connections:
- net +5V: now also U?.15 (Vin)
- net GND: now also RFID?.6 (GND), U?.17 (GND)
- net at R?.2: now also U?.28 (D2)
- net at Q?.3 (C), R?.1: now also R?.1 (x3)
- net at R?.2: now also U?.27 (D3)
- net at R?.2: now also U?.20 (D8)
- new net: RFID?.8 (3V3), U?.16 (3V3)
- new net: RFID?.3 (MOSI), U?.21 (D7)
- new net: RFID?.4 (MISO), U?.22 (D6)
- new net: RFID?.2 (SCK), U?.23 (D5)
- new net: RFID?.7 (RST), U?.29 (D1)
- new net: RFID?.1 (SDA), U?.30 (D0)
- new net: D?.1 (RED_ANODE), R?.2
- new net: D?.3 (BLUE_ANODE), R?.2
- new net: D?.4 (GREEN_ANODE), R?.2
Other:
- moved on the sheet: D?, Q?, R?

Commit message: minor changes
Parts:
- gave numbers to parts that had none: 22
Connections:
- no-connect marks 0 -> 17

Commit message: starting board design for magic stick
Parts:
- D1, D2: footprint (none) -> LEDs:LED-RGB-5MM_Common_Cathode
- Q1, Q2, Q3, Q4, Q5, Q6: footprint (none) -> TO_SOT_Packages_THT:TO-92_Inline_Narrow_Oval
- R1, R10, R11, R12, R2, R3, R4, R5, R6, R7, R8, R9: footprint (none) -> Resistors_ThroughHole:Resistor_Horizontal_RM10mm
- RFID1: footprint (none) -> Pin_Headers:Pin_Header_Straight_1x08
- U1: footprint (none) -> nodemcu:NodeMCU_Amica_R2
Changed lines of the file:
@@
 F 0 "D1" H 5400 3900 50  0000 C CNN
 F 1 "LED_RCBG" H 5400 3200 50  0000 C CNN
-F 2 "" H 5400 3500 50  0000 C CNN
+F 2 "LEDs:LED-RGB-5MM_Common_Cathode" H 5400 3500 50  0001 C CNN
 F 3 "" H 5400 3500 50  0000 C CNN
 	1    5400 3550
@@
 F 0 "R4" V 5780 2550 50  0000 C CNN
 F 1 "1k" V 5700 2550 50  0000 C CNN
-F 2 "" V 5630 2550 50  0000 C CNN
+F 2 "Resistors_ThroughHole:Resistor_Horizontal_RM10mm" V 5630 2550 50  0001 C CNN
 F 3 "" H 5700 2550 50  0000 C CNN
 	1    5700 2550
@@
 F 0 "R1" V 4080 2900 50  0000 C CNN
 F 1 "1k" V 4000 2900 50  0000 C CNN
-F 2 "" V 3930 2900 50  0000 C CNN
+F 2 "Resistors_ThroughHole:Resistor_Horizontal_RM10mm" V 3930 2900 50  0001 C CNN
 F 3 "" H 4000 2900 50  0000 C CNN
 	1    4000 2900
@@
 F 0 "R5" V 5930 3350 50  0000 C CNN
 F 1 "32" V 5850 3350 50  0000 C CNN
-F 2 "" V 5780 3350 50  0000 C CNN
+F 2 "Resistors_ThroughHole:Resistor_Horizontal_RM10mm" V 5780 3350 50  0001 C CNN
 F 3 "" H 5850 3350 50  0000 C CNN
 	1    5850 3350
@@
 F 0 "R6" V 5930 3550 50  0000 C CNN
 F 1 "21" V 5850 3550 50  0000 C CNN
-F 2 "" V 5780 3550 50  0000 C CNN
+F 2 "Resistors_ThroughHole:Resistor_Horizontal_RM10mm" V 5780 3550 50  0001 C CNN
 F 3 "" H 5850 3550 50  0000 C CNN
 	1    5850 3550
@@
 F 0 "R7" V 5930 3750 50  0000 C CNN
 F 1 "21" V 5850 3750 50  0000 C CNN
-F 2 "" V 5780 3750 50  0000 C CNN
+F 2 "Resistors_ThroughHole:Resistor_Horizontal_RM10mm" V 5780 3750 50  0001 C CNN
 F 3 "" H 5850 3750 50  0000 C CNN
 	1    5850 3750
@@
 F 0 "R11" V 6030 2900 50  0000 C CNN
 F 1 "1k" V 5950 2900 50  0000 C CNN
-F 2 "" V 5880 2900 50  0000 C CNN
+F 2 "Resistors_ThroughHole:Resistor_Horizontal_RM10mm" V 5880 2900 50  0001 C CNN
 F 3 "" H 5950 2900 50  0000 C CNN
 	1    5950 2900
@@
 F 0 "R12" V 6280 3150 50  0000 C CNN
 F 1 "1k" V 6200 3150 50  0000 C CNN
-F 2 "" V 6130 3150 50  0000 C CNN
+F 2 "Resistors_ThroughHole:Resistor_Horizontal_RM10mm" V 6130 3150 50  0001 C CNN
 F 3 "" H 6200 3150 50  0000 C CNN
 	1    6200 3150
@@
 F 0 "R2" V 4330 3100 50  0000 C CNN
 F 1 "1k" V 4250 3100 50  0000 C CNN
-F 2 "" V 4180 3100 50  0000 C CNN
+F 2 "Resistors_ThroughHole:Resistor_Horizontal_RM10mm" V 4180 3100 50  0001 C CNN
 F 3 "" H 4250 3100 50  0000 C CNN
 	1    4250 3100
@@
 F 0 "R3" V 4530 3350 50  0000 C CNN
 F 1 "1k" V 4450 3350 50  0000 C CNN
-F 2 "" V 4380 3350 50  0000 C CNN
+F 2 "Resistors_ThroughHole:Resistor_Horizontal_RM10mm" V 4380 3350 50  0001 C CNN
 F 3 "" H 4450 3350 50  0000 C CNN
 	1    4450 3350
@@
 F 0 "Q3" H 5100 3400 50  0000 R CNN
 F 1 "2N2222" H 5400 3300 50  0000 R CNN
-F 2 "" H 5000 3450 50  0000 C CNN
+F 2 "TO_SOT_Packages_THT:TO-92_Inline_Narrow_Oval" H 5000 3450 50  0001 C CNN
 F 3 "" H 4800 3350 50  0000 C CNN
 	1    4800 3350
@@
 F 0 "Q1" H 4650 2950 50  0000 R CNN
 F 1 "2N2222" H 4950 2850 50  0000 R CNN
-F 2 "" H 4550 3000 50  0000 C CNN
+F 2 "TO_SOT_Packages_THT:TO-92_Inline_Narrow_Oval" H 4550 3000 50  0001 C CNN
 F 3 "" H 4350 2900 50  0000 C CNN
 	1    4350 2900
@@
 F 0 "Q2" H 4900 3150 50  0000 R CNN
 F 1 "2N2222" H 5200 3050 50  0000 R CNN
-F 2 "" H 4800 3200 50  0000 C CNN
+F 2 "TO_SOT_Packages_THT:TO-92_Inline_Narrow_Oval" H 4800 3200 50  0001 C CNN
 F 3 "" H 4600 3100 50  0000 C CNN
 	1    4600 3100
@@
 F 0 "Q6" H 6850 3200 50  0000 R CNN
 F 1 "2N2907" H 7150 3100 50  0000 R CNN
-F 2 "" H 6750 3250 50  0000 C CNN
+F 2 "TO_SOT_Packages_THT:TO-92_Inline_Narrow_Oval" H 6750 3250 50  0001 C CNN
 F 3 "" H 6550 3150 50  0000 C CNN
 	1    6550 3150
@@
 F 0 "Q4" H 6350 2600 50  0000 R CNN
 F 1 "2N2907" H 6650 2500 50  0000 R CNN
-F 2 "" H 6250 2650 50  0000 C CNN
+F 2 "TO_SOT_Packages_THT:TO-92_Inline_Narrow_Oval" H 6250 2650 50  0001 C CNN
 F 3 "" H 6050 2550 50  0000 C CNN
 	1    6050 2550
@@
 F 0 "Q5" H 6600 2950 50  0000 R CNN
 F 1 "2N2907" H 6900 2850 50  0000 R CNN
-F 2 "" H 6500 3000 50  0000 C CNN
+F 2 "TO_SOT_Packages_THT:TO-92_Inline_Narrow_Oval" H 6500 3000 50  0001 C CNN
 F 3 "" H 6300 2900 50  0000 C CNN
 	1    6300 2900
@@
 F 0 "U1" H 2200 4200 50  0000 C CNN
 F 1 "NodeMCU_Amica_R2" H 2200 2550 50  0000 C CNN
-F 2 "" H 2450 3400 50  0000 C CNN
+F 2 "nodemcu:NodeMCU_Amica_R2" H 2450 3400 50  0001 C CNN
 F 3 "" H 2450 3400 50  0000 C CNN
 	1    2200 3400
@@
 F 0 "RFID1" H 3100 1600 60  0000 C CNN
 F 1 "RFID-RC522" H 3100 1100 60  0000 C CNN
-F 2 "" H 3100 1600 60  0000 C CNN
+F 2 "Pin_Headers:Pin_Header_Straight_1x08" H 3100 1600 60  0001 C CNN
 F 3 "" H 3100 1600 60  0000 C CNN
 	1    3100 1100
@@
 F 0 "D2" H 5400 4750 50  0000 C CNN
 F 1 "LED_RCBG" H 5400 4050 50  0000 C CNN
-F 2 "" H 5400 4350 50  0000 C CNN
+F 2 "LEDs:LED-RGB-5MM_Common_Cathode" H 5400 4350 50  0001 C CNN
 F 3 "" H 5400 4350 50  0000 C CNN
 	1    5400 4400
@@
 F 0 "R8" V 5930 4200 50  0000 C CNN
 F 1 "32" V 5850 4200 50  0000 C CNN
-F 2 "" V 5780 4200 50  0000 C CNN
+F 2 "Resistors_ThroughHole:Resistor_Horizontal_RM10mm" V 5780 4200 50  0001 C CNN
 F 3 "" H 5850 4200 50  0000 C CNN
 	1    5850 4200
@@
 F 0 "R9" V 5930 4400 50  0000 C CNN
 F 1 "21" V 5850 4400 50  0000 C CNN
-F 2 "" V 5780 4400 50  0000 C CNN
+F 2 "Resistors_ThroughHole:Resistor_Horizontal_RM10mm" V 5780 4400 50  0001 C CNN
 F 3 "" H 5850 4400 50  0000 C CNN
 	1    5850 4400
@@
 F 0 "R10" V 5930 4600 50  0000 C CNN
 F 1 "21" V 5850 4600 50  0000 C CNN
-F 2 "" V 5780 4600 50  0000 C CNN
+F 2 "Resistors_ThroughHole:Resistor_Horizontal_RM10mm" V 5780 4600 50  0001 C CNN
 F 3 "" H 5850 4600 50  0000 C CNN
 	1    5850 4600

Commit message: pcb for magic stick
Connections:
- net GND: now also D2.2 (COMMON_CATHODE), U1.14 (GND)
- net +3V3: now reaches U1.25 (3V3)
- no-connect marks 17 -> 15
Changed lines of the file:
@@
 NoConn ~ 1750 3800
 NoConn ~ 1750 3900
-NoConn ~ 1750 4000
 NoConn ~ 2650 3900
 NoConn ~ 2650 3800
 NoConn ~ 2650 3100
-NoConn ~ 2650 3200
 NoConn ~ 2650 3300
 NoConn ~ 1750 2700
@@
 Connection ~ 6650 3750
 Wire Wire Line
-	5150 4400 4900 4400
+	4900 4400 4900 3550
 Wire Wire Line
-	4900 4400 4900 3550
+	5100 4400 4900 4400
+$Comp
+L GND #PWR?
+U 1 1 5777E291
+P 1500 3950
+F 0 "#PWR?" H 1500 3700 50  0001 C CNN
+F 1 "GND" H 1500 3800 50  0000 C CNN
+F 2 "" H 1500 3950 50  0000 C CNN
+F 3 "" H 1500 3950 50  0000 C CNN
+	1    1500 3950
+	1    0    0    1
+$EndComp
+Wire Wire Line
+	1500 4000 1750 4000
+$Comp
+L +3.3V #PWR?
+U 1 1 5777E9C9
+P 3400 4100
+F 0 "#PWR?" H 3400 3950 50  0001 C CNN
+F 1 "+3.3V" H 3400 4240 50  0000 C CNN
+F 2 "" H 3400 4100 50  0000 C CNN
+F 3 "" H 3400 4100 50  0000 C CNN
+	1    3400 4100
+	1    0    0    -1
+$EndComp
+$Comp
+L +3.3V #PWR?
+U 1 1 5777EA09
+P 2800 3200
+F 0 "#PWR?" H 2800 3050 50  0001 C CNN
+F 1 "+3.3V" H 2800 3340 50  0000 C CNN
+F 2 "" H 2800 3200 50  0000 C CNN
+F 3 "" H 2800 3200 50  0000 C CNN
+	1    2800 3200
+	1    0    0    -1
+$EndComp
+Wire Wire Line
+	2650 3200 2800 3200
+Wire Wire Line
+	1500 4000 1500 3950
 $EndSCHEMATC

Commit message: magic stick updates
Connections:
- net GND: now also U1.10 (GND), U1.24 (GND)
- no-connect marks 15 -> 14
Changed lines of the file:
@@
 NoConn ~ 1750 3400
 NoConn ~ 1750 3500
-NoConn ~ 1750 3600
 NoConn ~ 1750 3700
 NoConn ~ 1750 3800
@@
 NoConn ~ 2650 3800
 NoConn ~ 2650 3100
-NoConn ~ 2650 3300
 NoConn ~ 1750 2700
 Wire Wire Line
@@
 	5100 4400 4900 4400
 $Comp
-L GND #PWR?
+L GND #PWR05
 U 1 1 5777E291
 P 1500 3950
-F 0 "#PWR?" H 1500 3700 50  0001 C CNN
+F 0 "#PWR05" H 1500 3700 50  0001 C CNN
 F 1 "GND" H 1500 3800 50  0000 C CNN
 F 2 "" H 1500 3950 50  0000 C CNN
@@
 	1500 4000 1750 4000
 $Comp
-L +3.3V #PWR?
+L +3.3V #PWR06
 U 1 1 5777E9C9
 P 3400 4100
-F 0 "#PWR?" H 3400 3950 50  0001 C CNN
+F 0 "#PWR06" H 3400 3950 50  0001 C CNN
 F 1 "+3.3V" H 3400 4240 50  0000 C CNN
 F 2 "" H 3400 4100 50  0000 C CNN
@@
 $EndComp
 $Comp
-L +3.3V #PWR?
+L +3.3V #PWR07
 U 1 1 5777EA09
 P 2800 3200
-F 0 "#PWR?" H 2800 3050 50  0001 C CNN
+F 0 "#PWR07" H 2800 3050 50  0001 C CNN
 F 1 "+3.3V" H 2800 3340 50  0000 C CNN
 F 2 "" H 2800 3200 50  0000 C CNN
@@
 Wire Wire Line
 	1500 4000 1500 3950
+NoConn ~ 3150 1700
+Wire Wire Line
+	2650 3300 2750 3300
+Wire Wire Line
+	1750 3600 1650 3600
+$Comp
+L GND #PWR08
+U 1 1 5778EBCC
+P 2750 3300
+F 0 "#PWR08" H 2750 3050 50  0001 C CNN
+F 1 "GND" H 2750 3150 50  0000 C CNN
+F 2 "" H 2750 3300 50  0000 C CNN
+F 3 "" H 2750 3300 50  0000 C CNN
+	1    2750 3300
+	1    0    0    -1
+$EndComp
+$Comp
+L GND #PWR09
+U 1 1 5778EC90
+P 1650 3600
+F 0 "#PWR09" H 1650 3350 50  0001 C CNN
+F 1 "GND" H 1650 3450 50  0000 C CNN
+F 2 "" H 1650 3600 50  0000 C CNN
+F 3 "" H 1650 3600 50  0000 C CNN
+	1    1650 3600
+	1    0    0    -1
+$EndComp
 $EndSCHEMATC

Commit message: initial mother board
Parts:
- added R13, R14, R15: 10k, Resistors_ThroughHole:Resistor_Horizontal_RM10mm, symbol R
Connections:
- net +5V: now also R13.2, R14.2, R15.2
- net at Q4.2 (B), R4.1: now also R13.1
- net at Q5.2 (B), R11.1: now also R14.1
- net at Q6.2 (B), R12.1: now also R15.1
Other:
- moved on the sheet: R11, R12, R4
Changed lines of the file:
@@
 L R R4
 U 1 1 577788C4
-P 5700 2550
-F 0 "R4" V 5780 2550 50  0000 C CNN
-F 1 "1k" V 5700 2550 50  0000 C CNN
-F 2 "Resistors_ThroughHole:Resistor_Horizontal_RM10mm" V 5630 2550 50  0001 C CNN
-F 3 "" H 5700 2550 50  0000 C CNN
-	1    5700 2550
+P 5350 2550
+F 0 "R4" V 5430 2550 50  0000 C CNN
+F 1 "1k" V 5350 2550 50  0000 C CNN
+F 2 "Resistors_ThroughHole:Resistor_Horizontal_RM10mm" V 5280 2550 50  0001 C CNN
+F 3 "" H 5350 2550 50  0000 C CNN
+	1    5350 2550
 	0    1    1    0
 $EndComp
@@
 L R R11
 U 1 1 57778DE3
-P 5950 2900
-F 0 "R11" V 6030 2900 50  0000 C CNN
-F 1 "1k" V 5950 2900 50  0000 C CNN
-F 2 "Resistors_ThroughHole:Resistor_Horizontal_RM10mm" V 5880 2900 50  0001 C CNN
-F 3 "" H 5950 2900 50  0000 C CNN
-	1    5950 2900
+P 5750 2900
+F 0 "R11" V 5830 2900 50  0000 C CNN
+F 1 "1k" V 5750 2900 50  0000 C CNN
+F 2 "Resistors_ThroughHole:Resistor_Horizontal_RM10mm" V 5680 2900 50  0001 C CNN
+F 3 "" H 5750 2900 50  0000 C CNN
+	1    5750 2900
 	0    1    1    0
 $EndComp
@@
 L R R12
 U 1 1 57778E6D
-P 6200 3150
-F 0 "R12" V 6280 3150 50  0000 C CNN
-F 1 "1k" V 6200 3150 50  0000 C CNN
-F 2 "Resistors_ThroughHole:Resistor_Horizontal_RM10mm" V 6130 3150 50  0001 C CNN
-F 3 "" H 6200 3150 50  0000 C CNN
-	1    6200 3150
+P 5950 3150
+F 0 "R12" V 6030 3150 50  0000 C CNN
+F 1 "1k" V 5950 3150 50  0000 C CNN
+F 2 "Resistors_ThroughHole:Resistor_Horizontal_RM10mm" V 5880 3150 50  0001 C CNN
+F 3 "" H 5950 3150 50  0000 C CNN
+	1    5950 3150
 	0    1    1    0
 $EndComp
@@
 NoConn ~ 1750 2700
 Wire Wire Line
-	4450 2550 5550 2550
-Wire Wire Line
 	4450 2550 4450 2700
 Wire Wire Line
@@
 Connection ~ 4450 3550
 Wire Wire Line
-	4700 2900 5800 2900
-Wire Wire Line
 	6400 2200 6400 2700
 Wire Wire Line
@@
 Wire Wire Line
 	6650 3750 6000 3750
-Wire Wire Line
-	6050 3150 4900 3150
 Connection ~ 4900 3550
 Wire Wire Line
@@
 Connection ~ 4700 3550
 Wire Wire Line
-	6150 2200 6650 2200
+	5700 2200 6650 2200
 Connection ~ 6150 2200
 Wire Wire Line
@@
 	1    0    0    -1
 $EndComp
+$Comp
+L R R13
+U 1 1 577945F3
+P 5700 2400
+F 0 "R13" V 5780 2400 50  0000 C CNN
+F 1 "10k" V 5700 2400 50  0000 C CNN
+F 2 "Resistors_ThroughHole:Resistor_Horizontal_RM10mm" V 5630 2400 50  0001 C CNN
+F 3 "" H 5700 2400 50  0000 C CNN
+	1    5700 2400
+	-1   0    0    1
+$EndComp
+Wire Wire Line
+	5700 2200 5700 2250
+Wire Wire Line
+	5500 2550 5850 2550
+Connection ~ 5700 2550
+Wire Wire Line
+	5200 2550 4450 2550
+Wire Wire Line
+	5600 2900 4700 2900
+Wire Wire Line
+	6100 2900 5900 2900
+Wire Wire Line
+	5800 3150 4900 3150
+Wire Wire Line
+	6350 3150 6100 3150
+$Comp
+L R R14
+U 1 1 57794DE8
+P 5850 2600
+F 0 "R14" V 5930 2600 50  0000 C CNN
+F 1 "10k" V 5850 2600 50  0000 C CNN
+F 2 "Resistors_ThroughHole:Resistor_Horizontal_RM10mm" V 5780 2600 50  0001 C CNN
+F 3 "" H 5850 2600 50  0000 C CNN
+	1    5850 2600
+	-1   0    0    1
+$EndComp
+$Comp
+L R R15
+U 1 1 57794E5F
+P 6050 2900
+F 0 "R15" V 6130 2900 50  0000 C CNN
+F 1 "10k" V 6050 2900 50  0000 C CNN
+F 2 "Resistors_ThroughHole:Resistor_Horizontal_RM10mm" V 5980 2900 50  0001 C CNN
+F 3 "" H 6050 2900 50  0000 C CNN
+	1    6050 2900
+	-1   0    0    1
+$EndComp
+Wire Wire Line
+	5850 2450 5850 2200
+Connection ~ 5850 2200
+Wire Wire Line
+	5850 2750 5900 2750
+Wire Wire Line
+	5900 2750 5900 2900
+Wire Wire Line
+	6050 2750 6050 2200
+Connection ~ 6050 2200
+Wire Wire Line
+	6050 3050 6200 3050
+Wire Wire Line
+	6200 3050 6200 3150
+Connection ~ 6200 3150
+Connection ~ 5900 2900
 $EndSCHEMATC

Commit message: fixed cc foot print; now need to redo motherboard :(
Parts:
- added SW1: SW_PUSH, Buttons_Switches_ThroughHole:SW_PUSH_SMALL, symbol SW_PUSH
Connections:
- net GND: now also SW1.1
- net at U1.4 (SD3): now also SW1.2
- no-connect marks 14 -> 13
Changed lines of the file:
@@
 	0    1    1    0
 $EndComp
-NoConn ~ 1750 3000
 NoConn ~ 1750 3100
 NoConn ~ 1750 3200
@@
 Connection ~ 6200 3150
 Connection ~ 5900 2900
+$Comp
+L SW_PUSH SW1
+U 1 1 57A5FF44
+P 1450 3000
+F 0 "SW1" H 1600 3110 50  0000 C CNN
+F 1 "SW_PUSH" H 1450 2920 50  0000 C CNN
+F 2 "Buttons_Switches_ThroughHole:SW_PUSH_SMALL" H 1450 3000 50  0001 C CNN
+F 3 "" H 1450 3000 50  0000 C CNN
+	1    1450 3000
+	1    0    0    -1
+$EndComp
+$Comp
+L GND #PWR?
+U 1 1 57A6014D
+P 1150 3000
+F 0 "#PWR?" H 1150 2750 50  0001 C CNN
+F 1 "GND" H 1150 2850 50  0000 C CNN
+F 2 "" H 1150 3000 50  0000 C CNN
+F 3 "" H 1150 3000 50  0000 C CNN
+	1    1150 3000
+	1    0    0    -1
+$EndComp
 $EndSCHEMATC
